Commit message: ping pong paddle xml add

File: src/gripper/ping_pong_paddle/exported/urdf/ping_pong_paddle.SLDASM.urdf (robot description, URDF)
Before this commit: robot ping_pong_paddle.SLDASM, 1 links, 0 joints
Links:
- link base_link: geometry collision mesh filename=base_link.STL; visual mesh filename=base_link.STL
